File: PCB/PicoQuantizer/PicoQuantizer.kicad_sch (KiCad schematic)
At the start: 49 parts, among them J1 Pitch in A, J2 Gate in A, J3 Pitch out A, J4 Pitch in B, J5 Gate in B, J6 Pitch out B, SW1 SW_SPDT, SW10 SW_SPDT, SW11 SW_SPDT, SW12 SW_SPDT, SW2 SW_SPDT, SW3 SW_SPDT, SW4 SW_SPDT, SW5 SW_SPDT, SW6 SW_SPDT, SW7 SW_SPDT, SW8 SW_SPDT, SW9 SW_SPDT, U1 TL072, U2 TL074, U3 MCP4911, U4 MCP4911

Commit message: code cleanup
Parts:
- removed D3, D4: D, symbol Device:D
- removed R10, R13, R4, R5, R8: 100k, symbol Device:R
- removed R3, R7: 33k, symbol Device:R
- added D10, D11, D12, D13, D14, D15, D16, D5, D6, D7, D8, D9: LED, symbol Device:LED
- added Q1, Q2: 2N3904, Package_TO_SOT_THT:TO-92_Inline, symbol Transistor_BJT:2N3904
- added R19, R21, R22: 100k, symbol Device:R
- added R20, R23: 10k, symbol Device:R
- added U5: LP2950-5.0_TO92, Package_TO_SOT_THT:TO-92_Inline, symbol Regulator_Linear:LP2950-5.0_TO92
- C1: value C -> 10nF
- R1: value 100k -> 10k
- R11: value 33k -> 10k
- R14: value 33k -> 100k
- R2, R6: value 100k -> 39k
Connections:
- net +3.3V is gone; now on net 5V: U3.6 (Vref), U4.6 (Vref)
- net +12V: now also U2.4 (V+), U5.3 (VI)
- net GND: now also J1.3 (SW), J2.3 (SW), SW1.3 (C), SW10.3 (C), SW11.3 (C), SW12.3 (C), SW2.3 (C), SW3.3 (C), SW4.3 (C), SW5.3 (C), SW6.3 (C), SW7.3 (C), SW8.3 (C), SW9.3 (C), U2.10 (+), U2.3 (+), D10.1 (K), D11.1 (K), D12.1 (K), D13.1 (K), D14.1 (K), D15.1 (K), D16.1 (K), D5.1 (K), D6.1 (K), D7.1 (K), D8.1 (K), D9.1 (K), R19.2, R21.2, U5.2 (GND); no longer R1.1, R11.1, R14.1
- net 5V: now reaches U1.6 (-)
- net 5V: now also U1.2 (-), U5.1 (VO)
- net at U1.7: now also R20.1
- net at R9.2: now also R11.1, R14.2, U2.2 (-); no longer U2.3 (+)
- net at R12.2: now also U2.9 (-), R22.2, R23.1; no longer U2.10 (+)
- net PITCH_B_IN: now reaches U2.8
- net PITCH_B_IN: now also A1.32 (GPIO27_ADC1), R23.2; no longer U2.9 (-)
- net PITCH_A_IN: now reaches R11.2
- net PITCH_A_IN: now also A1.31 (GPIO26_ADC0), U2.1
- net at SW4.1 (A): now also D8.2 (A)
- net NOTE_SEL_04: now reaches SW4.2 (B)
- net NOTE_SEL_04: now also A1.5 (GPIO3)
- net at C1.1, J2.1 (SIG), J5.3 (SW): no longer R1.2
- net at SW7.1 (A): now also D11.2 (A)
- net NOTE_SEL_07: now reaches SW7.2 (B)
- net NOTE_SEL_07: now also A1.9 (GPIO6)
- net at SW8.1 (A): now also D12.2 (A)
- net NOTE_SEL_08: now reaches SW8.2 (B)
- net NOTE_SEL_08: now also A1.10 (GPIO7)
- net -12V: now reaches U2.11 (V-)
- net -12V: now also R14.1, R22.1
- net at SW5.1 (A): now also D9.2 (A)
- net NOTE_SEL_05: now reaches SW5.2 (B)
- net NOTE_SEL_05: now also A1.6 (GPIO4)
- net NOTE_SEL_01: now reaches A1.1 (GPIO0)
- net NOTE_SEL_01: now also SW1.2 (B)
- net NOTE_SEL_09: now reaches A1.11 (GPIO8)
- net NOTE_SEL_09: now also SW9.2 (B)
- net NOTE_SEL_10: now reaches A1.12 (GPIO9)
- net NOTE_SEL_10: now also SW10.2 (B)
- net NOTE_SEL_11: now reaches A1.14 (GPIO10)
- net NOTE_SEL_11: now also SW11.2 (B)
- net NOTE_SEL_12: now reaches A1.15 (GPIO11)
- net NOTE_SEL_12: now also SW12.2 (B)
- net NOTE_SEL_02: now reaches A1.2 (GPIO1)
- net NOTE_SEL_02: now also SW2.2 (B)
- net GATE_A: now reaches A1.26 (GPIO20)
- net GATE_A: now also Q1.1 (E), R19.1
- net GATE_B: now reaches A1.27 (GPIO21)
- net GATE_B: now also Q2.1 (E), R21.1
- net +3V3: now reaches A1.36 (3V3)
- net +3V3: now also Q1.3 (C), Q2.3 (C)
- net NOTE_SEL_03: now reaches A1.4 (GPIO2)
- net NOTE_SEL_03: now also SW3.2 (B)
- net NOTE_SEL_06: now reaches A1.7 (GPIO5)
- net NOTE_SEL_06: now also SW6.2 (B)
- net at SW11.1 (A): now also D15.2 (A)
- net at SW2.1 (A): now also D6.2 (A)
- net at SW1.1 (A): now also D5.2 (A)
- net at SW12.1 (A): now also D16.2 (A)
- net at SW10.1 (A): now also D14.2 (A)
- net at SW6.1 (A): now also D10.2 (A)
- net at SW9.1 (A): now also D13.2 (A)
- net at U1.1: now also R1.1
- net at SW3.1 (A): now also D7.2 (A)
- new net: Q2.2 (B), R20.2
- new net: Q1.2 (B), R1.2
Other:
- note added: "/10 divider, offsets voltage up above 0, and inverts it essentially keeps it 0V to 3.3V"
- note added: "2x amplifier"
- note added: "Gate to trigger converter, or just trigger input"
- moved on the sheet: C2, D2, J1, J3, J4, J6, R12, R15, R16, R17, R18, R6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
